File: PCB/HexKey60.kicad_pcb (KiCad board)
At the start: 2 copper layers, 321.8 x 112.3 mm, 205 parts, among them SW1 SW_Push, SW10 SW_Push, SW11 SW_Push, SW12 SW_Push, SW13 SW_Push, SW14 SW_Push, SW15 SW_Push, SW16 SW_Push, SW17 SW_Push, SW18 SW_Push, SW19 SW_Push, SW2 SW_Push, SW20 SW_Push, SW21 SW_Push, SW22 SW_Push, SW23 SW_Push, SW24 SW_Push, SW25 SW_Push, SW26 SW_Push, SW27 SW_Push, SW28 SW_Push, SW29 SW_Push, SW3 SW_Push, SW30 SW_Push, SW31 SW_Push, SW32 SW_Push, SW33 SW_Push, SW34 SW_Push, SW35 SW_Push, SW36 SW_Push, SW37 SW_Push, SW38 SW_Push, SW39 SW_Push, SW4 SW_Push, SW40 SW_Push, SW41 SW_Push, SW42 SW_Push, SW43 SW_Push, SW44 SW_Push, SW45 SW_Push, SW46 SW_Push, SW47 SW_Push, SW48 SW_Push, SW49 SW_Push, SW5 SW_Push, SW50 SW_Push, SW51 SW_Push, SW52 SW_Push, SW53 SW_Push, SW54 SW_Push, SW55 SW_Push, SW56 SW_Push, SW57 SW_Push, SW58 SW_Push, SW59 SW_Push, SW6 SW_Push, SW60 SW_Push, SW61 SW_Push, SW62 SW_Push, SW63 SW_Push, SW64 SW_Push, SW65 SW_Push, SW66 SW_Push, SW67 SW_Push, SW68 SW_Push, SW7 SW_Push, SW8 SW_Push, SW9 SW_Push

Commit message: Add files via upload
Parts:
- added P1: USB_C_Plug_USB2.0, usbc:usbc board, F.Cu at (278.9, 36.0)
- SW1, SW10, SW11, SW12, SW13, SW14, SW15, SW16, SW17, SW18, SW19, SW2, SW20, SW21, SW22, SW23, SW24, SW25, SW26, SW27, SW28, SW29, SW3, SW30, SW31, SW32, SW33, SW34, SW35, SW36, SW37, SW38, SW39, SW4, SW40, SW41, SW42, SW43, SW44, SW45, SW46, SW47, SW48, SW49, SW5, SW50, SW51, SW52, SW53, SW54, SW55, SW56, SW57, SW58, SW59, SW6, SW60, SW61, SW62, SW63, SW64, SW65, SW66, SW67, SW68, SW7, SW8, SW9: footprint Button_Switch_Keyboard:SW_Cherry_MX_1.00u_Plate -> Button_Switch_Keyboard:SW_Cherry_MX_1.00u_PCB
Routing:
- net Net-(D100-VDD): track 1352.3 -> 1406.1 mm, vias 70 -> 78
- net Net-(D100-VSS): track 1736.0 -> 1787.9 mm, vias 63 -> 64
- net Net-(A1-GPIO3): track 421.2 -> 441.6 mm, vias 1 -> 5
- net Net-(A1-GPIO2): track 403.2 -> 419.5 mm, vias 6 -> 8
- net /col4: track 124.9 -> 136.9 mm, vias 12 -> 13
- net Net-(A1-GPIO0): track 648.7 -> 659.0 mm, vias 3 -> 4
- net Net-(A1-GPIO1): track 435.5 -> 444.4 mm
- net /col8: track 213.0 -> 221.8 mm
- net Net-(A1-VBUS): track 473.1 -> 481.8 mm, vias 5 -> 6
- net Net-(D98-DOUT): track 40.7 -> 49.2 mm
- net Net-(D82-DOUT): track 51.9 -> 59.2 mm, vias 6 -> 4
- net Net-(D134-DOUT): track 61.6 -> 68.8 mm
- net /col9: track 225.8 -> 231.1 mm
- net /col12: track 349.5 -> 353.7 mm
- net Net-(A1-GPIO4): track 395.5 -> 398.8 mm
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
Commit message: Add files via upload
Connections:
- net Net-(D100-VSS) renamed GND
Routing:
- added copper zone on B.Cu, net GND
Other:
- board text added: "Made By HexFud"
- board text added: "Thanks to"
